Commit message: Add diff_drive_example.

File: pca9685_ros2_control_example/bringup/description/description.urdf.xacro (robot description, xacro)
@@ -14,4 +14,7 @@
       <command_interface name="velocity"/>
     </joint>
+    <joint name="joint_3">
+      <command_interface name="velocity"/>
+    </joint>
   </ros2_control>
 </robot>
