Commit message: Add clamp command.

File: pca9685_ros2_control_example/description/description.urdf.xacro (robot description, xacro)
@@ -17,4 +17,10 @@
       <command_interface name="velocity"/>
     </joint>
+    <joint name="joint_4">
+      <command_interface name="velocity"/>
+    </joint>
+    <joint name="joint_5">
+      <command_interface name="velocity"/>
+    </joint>
   </ros2_control>
 </robot>

Commit message: Remove unneccesary things.

File: pca9685_ros2_control_example/description/description.urdf.xacro (robot description, xacro)
@@ -5,20 +5,4 @@
       <plugin>pca9685_hardware_interface/Pca9685SystemHardware</plugin>
     </hardware>
-    <joint name="joint_0">
-      <command_interface name="velocity"/>
-      <state_interface name="velocity"/>
-    </joint>
-    <joint name="joint_1">
-      <command_interface name="velocity"/>
-      <state_interface name="velocity"/>
-    </joint>
-    <joint name="joint_2">
-      <command_interface name="velocity"/>
-      <state_interface name="velocity"/>
-    </joint>
-    <joint name="joint_3">
-      <command_interface name="velocity"/>
-      <state_interface name="velocity"/>
-    </joint>
     <joint name="joint_4">
       <command_interface name="velocity"/>

Commit message: Update.

File: pca9685_ros2_control_example/description/description.urdf.xacro (robot description, xacro)
@@ -5,4 +5,20 @@
       <plugin>pca9685_hardware_interface/Pca9685SystemHardware</plugin>
     </hardware>
+    <joint name="joint_0">
+      <command_interface name="velocity"/>
+      <state_interface name="velocity"/>
+    </joint>
+    <joint name="joint_1">
+      <command_interface name="velocity"/>
+      <state_interface name="velocity"/>
+    </joint>
+    <joint name="joint_2">
+      <command_interface name="velocity"/>
+      <state_interface name="velocity"/>
+    </joint>
+    <joint name="joint_3">
+      <command_interface name="velocity"/>
+      <state_interface name="velocity"/>
+    </joint>
     <joint name="joint_4">
       <command_interface name="velocity"/>
